File: control.kicad_sch (KiCad schematic)
At the start: 43 parts, among them J6 BM03B-SRSS-TB, J7 TC2030-NL, J8 TYPE-C16PIN, SW2 KMR2, SW3 KMR2, U12 W25Q128JVS, U4 USBLC6-2SC6, U5 RP2350A, U6 NCP1117ST33T3G, Y1 ABM8-272-T3

Commit message: made some changes
Parts:
- added U14: ESP32-C3-MINI-1, Espressif:ESP32-C3-MINI-1, symbol Espressif:ESP32-C3-MINI-1
Connections:
- new net: U14.1 (GND), U14.11 (GND), U14.14 (GND), U14.2 (GND), U14.36 (GND), U14.37 (GND), U14.38 (GND), U14.39 (GND), U14.40 (GND), U14.41 (GND), U14.42 (GND), U14.43 (GND), U14.44 (GND), U14.45 (GND), U14.46 (GND), U14.47 (GND), U14.48 (GND), U14.49 (GND), U14.50 (GND), U14.51 (GND), U14.52 (GND), U14.53 (GND)
Changed lines of the file:
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@@
 	(label "QSPI_SDO"
 		(at 167.64 95.25 0)
+		(fields_autoplaced yes)
 		(effects
 			(font
@@
 	(label "QSPI_SCLK"
 		(at 167.64 92.71 0)
+		(fields_autoplaced yes)
 		(effects
 			(font
@@
 	(label "QSPI_SD2"
 		(at 167.64 100.33 0)
+		(fields_autoplaced yes)
 		(effects
 			(font
@@
 	(label "QSPI_SD1"
 		(at 167.64 97.79 0)
+		(fields_autoplaced yes)
 		(effects
 			(font
@@
 	(label "QSPI_SD3"
 		(at 167.64 102.87 0)
+		(fields_autoplaced yes)
 		(effects
 			(font
@@
 					(unit 1)
 				)
+			)
+		)
+	)
+	(symbol
+		(lib_id "Espressif:ESP32-C3-MINI-1")
+		(at 246.38 49.53 0)
+		(unit 1)
+		(exclude_from_sim no)
+		(in_bom yes)
+		(on_board yes)
+		(dnp no)
+		(fields_autoplaced yes)
+		(property "Reference" "U14"
+			(at 248.5741 19.05 0)
+			(effects
+				(font
+					(size 1.27 1.27)
+				)
+				(justify left)
+			)
+		)
+		(property "Value" "ESP32-C3-MINI-1"
+			(at 248.5741 21.59 0)
+			(effects
+				(font
+					(size 1.27 1.27)
+				)
+				(justify left)
+			)
+		)
+		(property "Footprint" "Espressif:ESP32-C3-MINI-1"
+			(at 246.38 85.09 0)
+			(effects
+				(font
+					(size 1.27 1.27)
+				)
+				(hide yes)
+			)
+		)
+		(property "Datasheet" "https://www.espressif.com/sites/default/files/documentation/esp32-c3-mini-1_datasheet_en.pdf"
+			(at 246.38 87.63 0)
+			(effects
+				(font
+					(size 1.27 1.27)
+				)
+				(hide yes)
+			)
+		)
+		(property "Description" "ESP32-C3-MINI-1 family is an ultra-low-power MCU-based SoC solution that supports 2.4 GHz Wi-Fi and Bluetooth®Low Energy (Bluetooth LE)."
+			(at 246.38 49.53 0)
+			(effects
+				(font
+					(size 1.27 1.27)
+				)
+				(hide yes)
+			)
+		)
+		(pin "14"
+		)
+		(pin "4"
+		)
+		(pin "1"
+		)
+		(pin "30"
+		)
+		(pin "10"
+		)
+		(pin "44"
+		)
+		(pin "43"
+		)
+		(pin "6"
+		)
+		(pin "7"
+		)
+		(pin "39"
+		)
+		(pin "8"
+		)
+		(pin "9"
+		)
+		(pin "34"
+		)
+		(pin "42"
+		)
+		(pin "11"
+		)
+		(pin "15"
+		)
+		(pin "31"
+		)
+		(pin "32"
+		)
+		(pin "33"
+		)
+		(pin "17"
+		)
+		(pin "51"
+		)
+		(pin "3"
+		)
+		(pin "26"
+		)
+		(pin "50"
+		)
+		(pin "12"
+		)
+		(pin "49"
+		)
+		(pin "27"
+		)
+		(pin "41"
+		)
+		(pin "28"
+		)
+		(pin "29"
+		)
+		(pin "48"
+		)
+		(pin "47"
+		)
+		(pin "52"
+		)
+		(pin "53"
+		)
+		(pin "16"
+		)
+		(pin "25"
+		)
+		(pin "46"
+		)
+		(pin "18"
+		)
+		(pin "45"
+		)
+		(pin "19"
+		)
+		(pin "13"
+		)
+		(pin "23"
+		)
+		(pin "24"
+		)
+		(pin "2"
+		)
+		(pin "38"
+		)
+		(pin "40"
+		)
+		(pin "37"
+		)
+		(pin "21"
+		)
+		(pin "20"
+		)
+		(pin "5"
+		)
+		(pin "22"
+		)
+		(pin "35"
+		)
+		(pin "36"
+		)
+		(instances
+			(project ""
+				(path "/e63e39d7-6ac0-4ffd-8aa3-1841a4541b55/76515553-b0fa-4a7a-9437-b8108a836ccb"
+					(reference "U14")
+					(unit 1)
+				)

Commit message: last modification for v2.0 before submitting order
Parts:
- removed U14: ESP32-C3-MINI-1, Espressif:ESP32-C3-MINI-1, symbol Espressif:ESP32-C3-MINI-1
- renumbered C15 to C14, C16 to C15, C17 to C16, C18 to C17, C19 to C18, C20 to C19, C21 to C20, C22 to C21, C23 to C22, C24 to C23, C25 to C24, C26 to C25, C27 to C26, C28 to C27, C43 to C28, D9 to D10, D10 to D9, R20 to R16, R21 to R17, R22 to R18, R24 to R19, R25 to R20, R16 to R21, R26 to R22, R27 to R23, R28 to R24, SW3 to SW2, SW2 to SW3, U4 to U5, U5 to U6, U12 to U7, U6 to U8
