File: imu.kicad_sch (KiCad schematic)
At the start: 5 parts, among them U7 LSM6DSM

Commit message: last modification for v2.0 before submitting order
Parts:
- U9: renamed from U7; value LSM6DSM -> LSM6DSOX
- renumbered R29 to R25, R30 to R26
Changed lines of the file:
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@@
 	(text "addr = 0"
 		(exclude_from_sim no)
-		(at 75.184 68.834 0)
+		(at 73.66 70.104 0)
 		(effects
 			(font
@@
 		(on_board yes)
 		(dnp no)
-		(property "Reference" "#PWR062"
+		(property "Reference" "#PWR057"
 			(at 110.49 64.77 0)
 			(effects
@@
 			(project "lil-G-electrical"
 				(path "/e63e39d7-6ac0-4ffd-8aa3-1841a4541b55/370f3da0-8967-4c65-8a1f-46aebfe65443"
-					(reference "#PWR062")
+					(reference "#PWR057")
 					(unit 1)
 				)
@@
 		(on_board yes)
 		(dnp no)
-		(property "Reference" "#PWR063"
+		(property "Reference" "#PWR058"
 			(at 96.52 101.6 0)
 			(effects
@@
 			(project "lil-G-electrical"
 				(path "/e63e39d7-6ac0-4ffd-8aa3-1841a4541b55/370f3da0-8967-4c65-8a1f-46aebfe65443"
-					(reference "#PWR063")
+					(reference "#PWR058")
 					(unit 1)
 				)
@@
 		(on_board yes)
 		(dnp no)
-		(property "Reference" "R30"
+		(property "Reference" "R26"
 			(at 68.326 75.692 0)
 			(effects
@@
 			(project "lil-G-electrical"
 				(path "/e63e39d7-6ac0-4ffd-8aa3-1841a4541b55/370f3da0-8967-4c65-8a1f-46aebfe65443"
-					(reference "R30")
+					(reference "R26")
 					(unit 1)
 				)
@@
 		(on_board yes)
 		(dnp no)
-		(property "Reference" "R29"
+		(property "Reference" "R25"
 			(at 60.706 75.692 0)
 			(effects
@@
 			(project "lil-G-electrical"
 				(path "/e63e39d7-6ac0-4ffd-8aa3-1841a4541b55/370f3da0-8967-4c65-8a1f-46aebfe65443"
-					(reference "R29")
+					(reference "R25")
 					(unit 1)
 				)
@@
 		(dnp no)
 		(fields_autoplaced yes)
-		(property "Reference" "U7"
+		(property "Reference" "U9"
 			(at 98.7141 91.44 0)
 			(effects
@@
 			)
 		)
-		(property "Value" "LSM6DSM"
+		(property "Value" "LSM6DSOX"
 			(at 98.7141 93.98 0)
 			(effects
@@
 			(project "lil-G-electrical"
 				(path "/e63e39d7-6ac0-4ffd-8aa3-1841a4541b55/370f3da0-8967-4c65-8a1f-46aebfe65443"
-					(reference "U7")
+					(reference "U9")
 					(unit 1)
 				)
@@
 		(on_board yes)
 		(dnp no)
-		(property "Reference" "#PWR061"
+		(property "Reference" "#PWR056"
 			(at 96.52 49.53 0)
 			(effects
@@
 			(project "lil-G-electrical"
 				(path "/e63e39d7-6ac0-4ffd-8aa3-1841a4541b55/370f3da0-8967-4c65-8a1f-46aebfe65443"
-					(reference "#PWR061")
-					(unit 1)
-				)
+					(reference "#PWR056")
+					(unit 1)
+				)
