File: lil-G-electrical.kicad_pcb (KiCad board)
At the start: 4 copper layers, 100 x 100 mm, 136 parts, among them J1 XT60-PW-M, J10 BM06B-SRSS-TB, J11 BM06B-SRSS-TB, J12 BM06B-SRSS-TB, J2 XT30-U-M, J3 XT60-PW-M, J4 BM04B-SRSS-TB, J5 BM03B-SRSS-TB, J6 BM03B-SRSS-TB, J7 TC2030-NL, J8 TYPE-C16PIN, J9 BM06B-SRSS-TB, Q1 40P30, SW1 5.8 ZSGT, SW2 KMR2, SW3 KMR2, U1 MCP1415, U10 A4950E, U11 A4950E, U12 W25Q128JVS, U2 TPS565208, U3 NCP1117ST33T3G, U4 USBLC6-2SC6, U5 RP2350A, U6 NCP1117ST33T3G, U7 LSM6DSM, U8 A4950E, U9 A4950E, Y1 ABM8-272-T3

Commit message: made some changes
Parts:
- added ?: , , F.Cu at (52.0, 48.4)
- added ?: , , F.Cu at (127.8, 48.7)
- added ?: , , F.Cu at (51.5, 123.5)
- moved D8 8.26 mm to (52.0, 103.3), turned to -90 degrees
- moved SW1 7.29 mm to (54.4, 110.0), turned to 90 degrees
- moved TP1 6.61 mm to (120.0, 118.9)
- moved R1 6.40 mm to (56.4, 115.8), turned to 180 degrees
- moved D3 5.17 mm to (54.4, 103.3), turned to -90 degrees
- moved TP2 5.04 mm to (126.7, 121.6)
- moved R25 4.50 mm to (51.4, 91.0)
- moved R13 4.50 mm to (61.6, 105.3), turned to 0 degrees
- moved R2 4.26 mm to (61.6, 102.7), turned to 0 degrees
- moved R5 3.98 mm to (61.6, 104.0), turned to 0 degrees
- moved TP3 3.83 mm to (123.3, 116.2)
- moved D1 3.03 mm to (56.8, 103.3), turned to -90 degrees
- moved SW3 2.50 mm to (52.2, 94.5)
- moved D10 2.40 mm to (55.5, 94.4)
- moved TP6 1.10 mm to (126.7, 113.5)
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Routing:
- net +5V: track 161.5 -> 174.6 mm
- net +3V3: track 329.4 -> 337.8 mm
- net /VBAT_FUSED: track 46.2 -> 52.6 mm
- net /PWR_EN: track 49.3 -> 45.9 mm
- net /rp2350a/~{RESET}: track 91.2 -> 88.9 mm
- net GND: track 90.6 -> 92.6 mm, vias 154 -> 166
- net Net-(D8-A): track 11.1 -> 9.86 mm
- net /I2C_SDA: track 52.7 -> 53.8 mm
- net /IMU_INT2: track 13.7 -> 14.5 mm
- net /rp2350a/SWCLK: track 55.8 -> 55.1 mm
- net /IMU_INT1: track 9.52 -> 10.2 mm
- net Net-(D3-A): track 8.07 -> 7.44 mm
- net /I2C_SCL: track 55.0 -> 55.6 mm
Other:
- board text added: "FUSE"
- board text added: "STATUS"

Commit message: last modification for v2.0 before submitting order
Parts:
- removed ? (x3): , 
- added TP6: 5001, TestPoint:TestPoint_Keystone_5000-5004_Miniature, F.Cu at (52.0, 48.4)
- added TP8: 5001, TestPoint:TestPoint_Keystone_5000-5004_Miniature, F.Cu at (127.8, 48.7)
- added TP9: 5001, TestPoint:TestPoint_Keystone_5000-5004_Miniature, F.Cu at (51.5, 123.5)
- renumbered C15 to C14, C16 to C15, C17 to C16, C18 to C17, C19 to C18, C20 to C19, C21 to C20, C22 to C21, C23 to C22, C24 to C23, C25 to C24, C26 to C25, C27 to C26, C28 to C27, C43 to C28, D9 to D10, D10 to D9, R14 to R10, R9 to R11, R10 to R12, R11 to R13, R12 to R14, R20 to R16, R21 to R17, R22 to R18, R24 to R19, R25 to R20, R16 to R21, R26 to R22, R27 to R23, R28 to R24, R29 to R25, R30 to R26, R31 to R27, R32 to R28, R33 to R29, R34 to R30, R35 to R31, R36 to R32, R37 to R33, R38 to R34, R39 to R35, R40 to R36, R41 to R37, R42 to R38, R13 to R9, SW3 to SW2, SW2 to SW3, TP3 to TP2, TP5 to TP3, TP6 to TP5, TP2 to TP7, U8 to U10, U9 to U11, U10 to U12, U11 to U13, U4 to U5, U5 to U6, U12 to U7, U6 to U8, U7 to U9
Routing:
- net /PWR_EN: track 45.9 -> 46.5 mm
- net GND: vias 166 -> 165
